Commit message: Get gazebo working

File: src/robot_description/description/robot_core.xacro (robot description, xacro)
@@ -20,9 +20,9 @@
         <parent link="base_link" />
         <child link="chassis" />
-        <origin xyz="-0.1 0 0" />
+        <origin xyz="0 0 0" />
     </joint>
     <link name="chassis">
         <visual>
-            <origin xyz="0.15 0 0.075" />
+            <origin xyz="0 0 0.075" />
             <geometry>
                 <box size="0.3 0.3 0.15" />
@@ -31,5 +31,5 @@
         </visual>
         <collision>
-            <origin xyz="0.15 0 0.075" />
+            <origin xyz="0 0 0.075" />
             <geometry>
                 <box size="0.3 0.3 0.15" />
@@ -37,5 +37,5 @@
         </collision>
         <xacro:inertial_box mass="0.5" x="0.3" y="0.3" z="0.15">
-            <origin xyz="0.15 0 0.075" rpy="0 0 0" />
+            <origin xyz="0 0 0.075" rpy="0 0 0" />
         </xacro:inertial_box>
     </link>
@@ -86,3 +86,80 @@
         </xacro:inertial_cylinder>
     </link>
+    <!-- DUMMY WHEELS AT FRONT AND BACK -->
+    <joint name="front_left_wheel_joint" type="fixed">
+        <parent link="base_link" />
+        <child link="front_left_wheel" />
+        <origin xyz="0.15 0.175 0" rpy="-${pi/2} 0 0" />
+        <axis xyz="0 0 1" />
+    </joint>
+    <link name="front_left_wheel">
+        <visual>
+            <geometry>
+                <cylinder radius="0.05" length="0.04" />
+            </geometry>
+            <material name="orange" />
+        </visual>
+        <collision>
+            <geometry>
+                <cylinder radius="0.0495" length="0.01" />
+            </geometry>
+        </collision>
+    </link>
+    <joint name="front_right_wheel_joint" type="fixed">
+        <parent link="base_link" />
+        <child link="front_right_wheel" />
+        <origin xyz="0.15 -0.175 0" rpy="${pi/2} 0 0" />
+        <axis xyz="0 0 -1" />
+    </joint>
+    <link name="front_right_wheel">
+        <visual>
+            <geometry>
+                <cylinder radius="0.05" length="0.04" />
+            </geometry>
+            <material name="orange" />
+        </visual>
+        <collision>
+            <geometry>
+                <cylinder radius="0.0495" length="0.01" />
+            </geometry>
+        </collision>
+    </link>
+    <joint name="back_left_wheel_joint" type="fixed">
+        <parent link="base_link" />
+        <child link="back_left_wheel" />
+        <origin xyz="-0.15 0.175 0" rpy="-${pi/2} 0 0" />
+        <axis xyz="0 0 1" />
+    </joint>
+    <link name="back_left_wheel">
+        <visual>
+            <geometry>
+                <cylinder radius="0.05" length="0.04" />
+            </geometry>
+            <material name="orange" />
+        </visual>
+        <collision>
+            <geometry>
+                <cylinder radius="0.0495" length="0.01" />
+            </geometry>
+        </collision>
+    </link>
+    <joint name="back_right_wheel_joint" type="fixed">
+        <parent link="base_link" />
+        <child link="back_right_wheel" />
+        <origin xyz="-0.15 -0.175 0" rpy="${pi/2} 0 0" />
+        <axis xyz="0 0 -1" />
+    </joint>
+    <link name="back_right_wheel">
+        <visual>
+            <geometry>
+                <cylinder radius="0.05" length="0.04" />
+            </geometry>
+            <material name="orange" />
+        </visual>
+        <collision>
+            <geometry>
+                <cylinder radius="0.0495" length="0.01" />
+            </geometry>
+        </collision>
+    </link>
 </robot>
