Commit message: Rename robot_description package due to ros2_control naming conflict. Setup gazebo for ros2_control

File: src/robot_tank_desc/description/gazebo_control.xacro (robot description, xacro)
@@ -6,6 +6,6 @@
             <left_joint>left_wheel_joint</left_joint>
             <right_joint>right_wheel_joint</right_joint>
-            <wheel_separation>0.35</wheel_separation>
-            <wheel_radius>0.05</wheel_radius>
+            <wheel_separation>0.245</wheel_separation>
+            <wheel_radius>0.0412</wheel_radius>
             <!-- Limits -->
             <max_linear_acceleration>5.0</max_linear_acceleration>

File: src/robot_tank_desc/description/robot_core.xacro (robot description, xacro)
@@ -33,5 +33,5 @@
             <geometry>
                 <!-- <box size="0.356 0.195 0.074" /> -->
-                <mesh filename="file://$(find robot_description)/stl/robot_frame.stl" scale="0.001 0.001 0.001" />
+                <mesh filename="file://$(find robot_tank_desc)/stl/robot_frame.stl" scale="0.001 0.001 0.001" />
             </geometry>
             <material name="yellow" />

Commit message: Add cameras to robot model

File: src/robot_tank_desc/description/gazebo_control.xacro (robot description, xacro)
@@ -24,25 +24,4 @@
             <joint_name>right_wheel_joint</joint_name>
         </plugin>
-        <plugin
-            filename="gz-sim-sensors-system"
-            name="gz::sim::systems::Sensors">
-            <render_engine>ogre2</render_engine>
-        </plugin>
-        <!-- <plugin
-        filename="gz-sim-physics-system"
-        name="gz::sim::systems::Physics">
-        </plugin>
-        <plugin
-        filename="gz-sim-user-commands-system"
-        name="gz::sim::systems::UserCommands">
-        </plugin>
-        <plugin
-        filename="gz-sim-scene-broadcaster-system"
-        name="gz::sim::systems::SceneBroadcaster">
-        </plugin>
-        <plugin
-        filename="gz-sim-imu-system"
-        name="gz::sim::systems::Imu">
-        </plugin> -->
     </gazebo>
 </robot>

File: src/robot_tank_desc/description/robot.urdf.xacro (robot description, xacro)
@@ -1,6 +1,11 @@
 <?xml version="1.0"?>
 <robot xmlns:xacro="http://www.ros.org/wiki/xacro" name="robot">
+    <xacro:arg name="sim_mode" default="false" />
     <xacro:include filename="robot_core.xacro" />
     <xacro:include filename="lidar.xacro" />
+    <xacro:include filename="cameras.xacro" />
+    <xacro:if value="$(arg sim_mode)">
+        <xacro:include filename="gz_plugins.xacro" />
+    </xacro:if>
     <!-- <xacro:include filename="gazebo_control.xacro" /> -->
     <xacro:include filename="ros2_control.xacro" />

File: src/robot_tank_desc/description/ros2_control.xacro (robot description, xacro)
@@ -1,28 +1,54 @@
 <?xml version="1.0"?>
 <robot xmlns:xacro="http://www.ros.org/wiki/xacro">
-    <ros2_control name="GazeboSystem" type="system">
-        <hardware>
-            <plugin>gz_ros2_control/GazeboSimSystem</plugin>
-        </hardware>
-        <joint name="left_wheel_joint">
-            <command_interface name="velocity">
-                <param name="min">-10</param>
-                <param name="max">10</param>
-            </command_interface>
-            <state_interface name="velocity"/>
-            <state_interface name="position"/>
-        </joint>
-        <joint name="right_wheel_joint">
-            <command_interface name="velocity">
-                <param name="min">-10</param>
-                <param name="max">10</param>
-            </command_interface>
-            <state_interface name="velocity"/>
-            <state_interface name="position"/>
-        </joint>
-    </ros2_control>
+    <xacro:unless value="$(arg sim_mode)">
+        <ros2_control name="RealRobot" type="system">
+            <hardware>
+                <plugin>diffdrive_rpi/DiffDriveRPI_TODO</plugin>
+            </hardware>
+            <joint name="left_wheel_joint">
+                <command_interface name="velocity">
+                    <param name="min">-10</param>
+                    <param name="max">10</param>
+                </command_interface>
+                <state_interface name="velocity"/>
+                <state_interface name="position"/>
+            </joint>
+            <joint name="right_wheel_joint">
+                <command_interface name="velocity">
+                    <param name="min">-10</param>
+                    <param name="max">10</param>
+                </command_interface>
+                <state_interface name="velocity"/>
+                <state_interface name="position"/>
+            </joint>
+        </ros2_control>
+    </xacro:unless>
+    <xacro:if value="$(arg sim_mode)">
+        <ros2_control name="GazeboSystem" type="system">
+            <hardware>
+                <plugin>gz_ros2_control/GazeboSimSystem</plugin>
+            </hardware>
+            <joint name="left_wheel_joint">
+                <command_interface name="velocity">
+                    <param name="min">-10</param>
+                    <param name="max">10</param>
+                </command_interface>
+                <state_interface name="velocity"/>
+                <state_interface name="position"/>
+            </joint>
+            <joint name="right_wheel_joint">
+                <command_interface name="velocity">
+                    <param name="min">-10</param>
+                    <param name="max">10</param>
+                </command_interface>
+                <state_interface name="velocity"/>
+                <state_interface name="position"/>
+            </joint>
+        </ros2_control>
+    </xacro:if>
     <gazebo>
         <plugin filename="libgz_ros2_control-system.so" name="gz_ros2_control::GazeboSimROS2ControlPlugin">
             <parameters>$(find robot_tank_desc)/config/controllers.yaml</parameters>
+            <parameters>$(find robot_tank_desc)/config/gz_ros2_control_use_sim.yaml</parameters>
         </plugin>
     </gazebo>
