Commit message: Update robot model to new smaller size

File: src/robot_tank_desc/description/cameras.xacro (robot description, xacro)
@@ -5,5 +5,5 @@
         <parent link="chassis" />
         <child link="camera_front_link" />
-        <origin xyz="0.178 0 0.025" rpy="0 0 0" />
+        <origin xyz="0.1305 0 0.025" rpy="0 0 0" />
     </joint>
     <link name="camera_front_link">
@@ -56,5 +56,5 @@
         <parent link="chassis" />
         <child link="camera_back_link" />
-        <origin xyz="-0.178 0 0.025" rpy="0 0 ${-pi}" />
+        <origin xyz="-0.1305 0 0.025" rpy="0 0 ${-pi}" />
     </joint>
     <link name="camera_back_link">

File: src/robot_tank_desc/description/robot_core.xacro (robot description, xacro)
@@ -20,17 +20,31 @@
         <color rgba="1 1 0 1"/>
     </material>
+    <xacro:macro name="robot_wheel">
+        <visual>
+            <geometry>
+                <cylinder radius="0.0411" length="0.05" />
+            </geometry>
+            <material name="orange" />
+        </visual>
+        <collision>
+            <geometry>
+                <cylinder radius="0.0411" length="0.05" />
+            </geometry>
+        </collision>
+    </xacro:macro>
     <link name="base_link">
     </link>
     <!-- CHASSIS LINK -->
+    <!-- Note 0.0206 is to offset the wheels onto the ground -->
     <joint name="chassis_joint" type="fixed">
         <parent link="base_link" />
         <child link="chassis" />
-        <origin xyz="0 0 0.066345" />
+        <origin xyz="0 0 ${0.066345 + 0.0206}" />
     </joint>
     <link name="chassis">
         <visual>
-            <origin xyz="0 -0.090 0" rpy="0 0 -${pi/2}" />
+            <origin xyz="0.0475 -0.090 0" rpy="0 0 -${pi/2}" />
             <geometry>
-                <!-- <box size="0.356 0.195 0.074" /> -->
+                <!-- <box size="0.261 0.195 0.074" /> -->
                 <mesh filename="file://$(find robot_tank_desc)/stl/robot_frame.stl" scale="0.001 0.001 0.001" />
             </geometry>
@@ -40,5 +54,5 @@
             <origin xyz="0 0 -0.037" />
             <geometry>
-                <box size="0.356 0.195 0.074" />
+                <box size="0.261 0.195 0.074" />
             </geometry>
         </collision>
@@ -53,5 +67,5 @@
         <parent link="base_link" />
         <child link="left_wheel" />
-        <origin xyz="0 0.1225 0" rpy="-${pi/2} 0 0" />
+        <origin xyz="0 0.1225 0.0206" rpy="-${pi/2} 0 0" />
         <axis xyz="0 0 1" />
     </joint>
@@ -76,5 +90,5 @@
         <parent link="base_link" />
         <child link="right_wheel" />
-        <origin xyz="0 -0.1225 0" rpy="${pi/2} 0 0" />
+        <origin xyz="0 -0.1225 0.0206" rpy="${pi/2} 0 0" />
         <axis xyz="0 0 -1" />
     </joint>
@@ -99,152 +113,72 @@
         <parent link="base_link" />
         <child link="front_left_bottom_wheel" />
-        <origin xyz="0.124 -0.1225 0" rpy="-${pi/2} 0 0" />
+        <origin xyz="0.0763 -0.1225 0.0206" rpy="-${pi/2} 0 0" />
         <axis xyz="0 0 1" />
     </joint>
     <link name="front_left_bottom_wheel">
-        <visual>
-            <geometry>
-                <cylinder radius="0.0411" length="0.05" />
-            </geometry>
-            <material name="orange" />
-        </visual>
-        <collision>
-            <geometry>
-                <cylinder radius="0.0411" length="0.05" />
-            </geometry>
-        </collision>
+        <xacro:robot_wheel />
     </link>
     <joint name="front_left_top_wheel_joint" type="fixed">
         <parent link="base_link" />
         <child link="front_left_top_wheel" />
-        <origin xyz="0.1705 -0.1225 0.058845" rpy="-${pi/2} 0 0" />
+        <origin xyz="0.1230 -0.1225 ${0.058845 + 0.0206}" rpy="-${pi/2} 0 0" />
         <axis xyz="0 0 1" />
     </joint>
     <link name="front_left_top_wheel">
-        <visual>
-            <geometry>
-                <cylinder radius="0.0411" length="0.05" />
-            </geometry>
-            <material name="orange" />
-        </visual>
-        <collision>
-            <geometry>
-                <cylinder radius="0.0411" length="0.05" />
-            </geometry>
-        </collision>
+        <xacro:robot_wheel />
     </link>
     <joint name="front_right_bottom_wheel_joint" type="fixed">
         <parent link="base_link" />
         <child link="front_right_bottom_wheel" />
-        <origin xyz="0.124 0.1225 0" rpy="-${pi/2} 0 0" />
+        <origin xyz="0.0763 0.1225 0.0206" rpy="-${pi/2} 0 0" />
         <axis xyz="0 0 -1" />
     </joint>
     <link name="front_right_bottom_wheel">
-        <visual>
-            <geometry>
-                <cylinder radius="0.0411" length="0.05" />
-            </geometry>
-            <material name="orange" />
-        </visual>
-        <collision>
-            <geometry>
-                <cylinder radius="0.0411" length="0.05" />
-            </geometry>
-        </collision>
+        <xacro:robot_wheel />
     </link>
     <joint name="front_right_top_wheel_joint" type="fixed">
         <parent link="base_link" />
         <child link="front_right_top_wheel" />
-        <origin xyz="0.1705 0.1225 0.058845" rpy="-${pi/2} 0 0" />
+        <origin xyz="0.1230 0.1225 ${0.058845 + 0.0206}" rpy="-${pi/2} 0 0" />
         <axis xyz="0 0 1" />
     </joint>
     <link name="front_right_top_wheel">
-        <visual>
-            <geometry>
-                <cylinder radius="0.0411" length="0.05" />
-            </geometry>
-            <material name="orange" />
-        </visual>
-        <collision>
-            <geometry>
-                <cylinder radius="0.0411" length="0.05" />
-            </geometry>
-        </collision>
+        <xacro:robot_wheel />
     </link>
     <joint name="back_left_bottom_wheel_joint" type="fixed">
         <parent link="base_link" />
         <child link="back_left_bottom_wheel" />
-        <origin xyz="-0.124 -0.1225 0" rpy="-${pi/2} 0 0" />
+        <origin xyz="-0.0763 -0.1225 0.0206" rpy="-${pi/2} 0 0" />
         <axis xyz="0 0 1" />
     </joint>
     <link name="back_left_bottom_wheel">
-        <visual>
-            <geometry>
-                <cylinder radius="0.0411" length="0.05" />
-            </geometry>
-            <material name="orange" />
-        </visual>
-        <collision>
-            <geometry>
-                <cylinder radius="0.0411" length="0.05" />
-            </geometry>
-        </collision>
+        <xacro:robot_wheel />
     </link>
     <joint name="back_left_top_wheel_joint" type="fixed">
         <parent link="base_link" />
         <child link="back_left_top_wheel" />
-        <origin xyz="-0.1705 -0.1225 0.058845" rpy="-${pi/2} 0 0" />
+        <origin xyz="-0.1230 -0.1225 ${0.058845 + 0.0206}" rpy="-${pi/2} 0 0" />
         <axis xyz="0 0 1" />
     </joint>
     <link name="back_left_top_wheel">
-        <visual>
-            <geometry>
-                <cylinder radius="0.0411" length="0.05" />
-            </geometry>
-            <material name="orange" />
-        </visual>
-        <collision>
-            <geometry>
-                <cylinder radius="0.0411" length="0.05" />
-            </geometry>
-        </collision>
+        <xacro:robot_wheel />
     </link>
-    <joint name="back_right_wheel_joint" type="fixed">
+    <joint name="back_right_bottom_wheel_joint" type="fixed">
         <parent link="base_link" />
-        <child link="back_right_wheel" />
-        <origin xyz="-0.124 0.1225 0" rpy="-${pi/2} 0 0" />
+        <child link="back_right_bottom_wheel" />
+        <origin xyz="-0.0763 0.1225 0.0206" rpy="-${pi/2} 0 0" />
         <axis xyz="0 0 -1" />
     </joint>
-    <link name="back_right_wheel">
-        <visual>
-            <geometry>
-                <cylinder radius="0.0411" length="0.05" />
-            </geometry>
-            <material name="orange" />
-        </visual>
-        <collision>
-            <geometry>
-                <cylinder radius="0.0411" length="0.05" />
-            </geometry>
-        </collision>
+    <link name="back_right_bottom_wheel">
+        <xacro:robot_wheel />
     </link>
     <joint name="back_right_top_wheel_joint" type="fixed">
         <parent link="base_link" />
         <child link="back_right_top_wheel" />
-        <origin xyz="-0.1705 0.1225 0.058845" rpy="-${pi/2} 0 0" />
+        <origin xyz="-0.1230 0.1225 ${0.058845 + 0.0206}" rpy="-${pi/2} 0 0" />
         <axis xyz="0 0 1" />
     </joint>
     <link name="back_right_top_wheel">
-        <visual>
-            <geometry>
-                <cylinder radius="0.0411" length="0.05" />
-            </geometry>
-            <material name="orange" />
-        </visual>
-        <collision>
-            <geometry>
-                <cylinder radius="0.0411" length="0.05" />
-            </geometry>
-        </collision>
+        <xacro:robot_wheel />
     </link>
 </robot>
