Commit message: Move lidar

File: src/robot_tank_desc/description/lidar.xacro (robot description, xacro)
@@ -4,5 +4,5 @@
         <parent link="chassis" />
         <child link="laser_frame" />
-        <origin xyz="0 0 0.05" rpy="0 0 0" />
+        <origin xyz="0.10525 ${0.02375 * 2.5} 0.132" rpy="0 0 0" />
     </joint>
     <link name="laser_frame">
@@ -21,4 +21,17 @@
             <origin xyz="0 0 0" rpy="0 0 0" />
         </xacro:inertial_cylinder>
+    </link>
+    <joint name="laser_rod_joint" type="fixed">
+        <parent link="chassis" />
+        <child link="laser_rod" />
+        <origin xyz="0.10525 ${0.02375 * 2.5} 0.05" rpy="0 0 0" />
+    </joint>
+    <link name="laser_rod">
+        <visual>
+            <geometry>
+                <cylinder radius="0.011" length="0.14" />
+            </geometry>
+            <material name="red" />
+        </visual>
     </link>
     <gazebo reference="laser_frame">

File: src/robot_tank_desc/description/robot_core.xacro (robot description, xacro)
@@ -34,4 +34,11 @@
     </xacro:macro>
     <link name="base_link">
+    </link>
+    <joint name="base_footprint_joint" type="fixed">
+        <parent link="base_link" />
+        <child link="base_footprint" />
+        <origin xyz="0 0 0" rpy="0 0 0" />
+    </joint>
+    <link name="base_footprint">
     </link>
     <!-- CHASSIS LINK -->

Commit message: Add fake stepper encoding using step count maths

File: src/robot_tank_desc/description/lidar.xacro (robot description, xacro)
@@ -4,5 +4,5 @@
         <parent link="chassis" />
         <child link="laser_frame" />
-        <origin xyz="0.10525 ${0.02375 * 2.5} 0.132" rpy="0 0 0" />
+         <origin xyz="0.10525 ${0.02375 * 2.5} 0.132" rpy="0 0 ${pi/2}" />
     </joint>
     <link name="laser_frame">
