Commit message: Tweak slam and nav2 params

File: src/robot_tank_desc/description/robot_core.xacro (robot description, xacro)
@@ -74,5 +74,6 @@
         <parent link="base_link" />
         <child link="left_wheel" />
-        <origin xyz="0 0.1225 0.0206" rpy="-${pi/2} 0 0" />
+        <!-- Note the wheel is offset on X to account for the center of gravity/turn radius being towards the back of the robot -->
+        <origin xyz="-0.05 0.1225 0.0206" rpy="-${pi/2} 0 0" />
         <axis xyz="0 0 1" />
     </joint>
@@ -97,5 +98,6 @@
         <parent link="base_link" />
         <child link="right_wheel" />
-        <origin xyz="0 -0.1225 0.0206" rpy="${pi/2} 0 0" />
+        <!-- Note the wheel is offset on X to account for the center of gravity/turn radius being towards the back of the robot -->
+        <origin xyz="-0.05 -0.1225 0.0206" rpy="${pi/2} 0 0" />
         <axis xyz="0 0 -1" />
     </joint>
